Commit message: dummy link added to urdf, to avoid warning

File: buggy_descripation/urdf/buggy_descripation.urdf (robot description, URDF)
Before this commit: robot buggy_descripation, 21 links, 20 joints
Links:
- added link dummy

Commit message: removed dummy link added to urdf, to avoid error

File: buggy_descripation/urdf/buggy_descripation.urdf (robot description, URDF)
Before this commit: robot buggy_descripation, 22 links, 20 joints
Links:
- removed link dummy

Commit message: Changes for wheels, new world and map added, changed scan list in config files. Mainly lidar name changed to laser even the STL files

File: buggy_descripation/urdf/buggy_descripation.urdf (robot description, URDF)
Before this commit: robot buggy_descripation, 22 links, 21 joints
Links:
- removed link dummy
- removed link lidar
- added link laser, mass 0.0887753797922069; collision mesh filename=package://buggy_descripation/meshes/laser.STL; visual mesh filename=package://buggy_descripation/meshes/laser.STL
Joints:
- removed joint dummy_joint
- joint lidar_joint: axis 0 0 0 -> 0 1 0; child lidar -> laser

Commit message: Navigation part ready, URDF problem needs to be fixed

File: buggy_descripation/urdf/buggy_descripation.urdf (robot description, URDF)
Before this commit: robot buggy_descripation, 21 links, 20 joints
Joints:
- joint lidar_joint: axis 0 1 0 -> 0 0 0; origin xyz=0 0.105 0 rpy=0 0 0 -> xyz=0 0.5 0 rpy=0 -1.5707963 1.5707963
