Commit message: laser_1 name changed to laser

File: buggy_description/urdf/buggy.xacro (robot description, xacro)
@@ -26,5 +26,5 @@
   </collision>
 </link>
-<link name="laser_1">
+<link name="laser">
   <inertial>
     <origin rpy="0 0 0" xyz="2.7755575615628914e-17 1.1102230246251565e-16 0.019476889152607244"/>
@@ -35,5 +35,5 @@
     <origin rpy="0 0 0" xyz="-0.09 -0.1745 -0.115"/>
     <geometry>
-      <mesh filename="package://buggy_description/meshes/laser_1.stl" scale="0.001 0.001 0.001"/>
+      <mesh filename="package://buggy_description/meshes/laser.stl" scale="0.001 0.001 0.001"/>
     </geometry>
     <material name="silver"/>
@@ -42,5 +42,5 @@
     <origin rpy="0 0 0" xyz="-0.09 -0.1745 -0.115"/>
     <geometry>
-      <mesh filename="package://buggy_description/meshes/laser_1.stl" scale="0.001 0.001 0.001"/>
+      <mesh filename="package://buggy_description/meshes/laser.stl" scale="0.001 0.001 0.001"/>
     </geometry>
   </collision>
@@ -169,5 +169,5 @@
   <origin rpy="0 0 0" xyz="0.09 0.1745 0.115"/>
   <parent link="base_link"/>
-  <child link="laser_1"/>
+  <child link="laser"/>
 </joint>
 <joint name="Rev2" type="continuous">
